File: examples/ESP32S3/Lilka_v2/src/context/apps/batt_test/module_resources/kicad_proj/test_battery/test_battery.kicad_sch (KiCad schematic)
At the start: 23 parts, among them J1 FUN, Q1 PN2222A, Q2 NMOS, Q3 NMOS, U1 PC817, U2 TL071, U3 INA219AxD

Commit message: chore example: виправлено схему модуля
Parts:
- added C2: 10u, symbol Device:C_Small
- added C3: 100n, symbol Device:C_Small
Connections:
- net GND: now also C2.2, C3.2
- net 9-12V renamed 12V
- net 12V: now also C2.1, C3.1
- net V_BAT + renamed BAT +1V5...8V4

Commit message: chore example: виправлення схеми
Parts:
- removed R10, R11: 100, symbol Device:R_Small
Connections:
- net at R8.2, R9.2: now also Q2.2 (G), Q3.2 (G)
Changed lines of the file:
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@@
 	(wire
 		(pts
-			(xy 180.34 115.57) (xy 189.23 115.57)
+			(xy 180.34 115.57) (xy 201.93 115.57)
 		)
 		(stroke
@@
 	(wire
 		(pts
-			(xy 195.58 130.81) (xy 213.36 130.81)
+			(xy 195.58 130.81) (xy 222.25 130.81)
 		)
 		(stroke
@@
 	(wire
 		(pts
-			(xy 218.44 130.81) (xy 222.25 130.81)
-		)
-		(stroke
-			(width 0)
-			(type default)
-		)
-	)
-	(wire
-		(pts
 			(xy 177.8 46.99) (xy 172.72 46.99)
 		)
@@
 		(pts
 			(xy 224.79 81.28) (xy 224.79 85.09)
-		)
-		(stroke
-			(width 0)
-			(type default)
-		)
-	)
-	(wire
-		(pts
-			(xy 194.31 115.57) (xy 201.93 115.57)
 		)
 		(stroke
@@
 	)
 	(symbol
-		(lib_id "Device:R_Small")
-		(at 191.77 115.57 90)
-		(unit 1)
-		(exclude_from_sim no)
-		(in_bom yes)
-		(on_board yes)
-		(dnp no)
-		(fields_autoplaced yes)
-		(property "Reference" "R10"
-			(at 191.77 110.49 90)
-			(effects
-				(font
-					(size 1.27 1.27)
-				)
-			)
-		)
-		(property "Value" "100"
-			(at 191.77 113.03 90)
-			(effects
-				(font
-					(size 1.27 1.27)
-				)
-			)
-		)
-		(property "Footprint" ""
-			(at 191.77 115.57 0)
-			(effects
-				(font
-					(size 1.27 1.27)
-				)
-				(hide yes)
-			)
-		)
-		(property "Datasheet" "~"
-			(at 191.77 115.57 0)
-			(effects
-				(font
-					(size 1.27 1.27)
-				)
-				(hide yes)
-			)
-		)
-		(property "Description" "Resistor, small symbol"
-			(at 191.77 115.57 0)
-			(effects
-				(font
-					(size 1.27 1.27)
-				)
-				(hide yes)
-			)
-		)
-		(pin "1"
-		)
-		(pin "2"
-		)
-		(instances
-			(project "test_battery"
-				(path "/21f56d4c-c23c-4f64-b5d5-a4783ab5b75c"
-					(reference "R10")
-					(unit 1)
-				)
-			)
-		)
-	)
-	(symbol
 		(lib_id "power:GND")
 		(at 224.79 96.52 0)
@@
 					(unit 1)
 				)
-			)
-		)
-	)
-	(symbol
-		(lib_id "Device:R_Small")
-		(at 215.9 130.81 90)
-		(unit 1)
-		(exclude_from_sim no)
-		(in_bom yes)
-		(on_board yes)
-		(dnp no)
-		(fields_autoplaced yes)
-		(property "Reference" "R11"
-			(at 215.9 125.73 90)
-			(effects
-				(font
-					(size 1.27 1.27)
-				)
-			)
-		)
-		(property "Value" "100"
-			(at 215.9 128.27 90)
-			(effects
-				(font
-					(size 1.27 1.27)
-				)
-			)
-		)
-		(property "Footprint" ""
-			(at 215.9 130.81 0)
-			(effects
-				(font
-					(size 1.27 1.27)
-				)
-				(hide yes)
-			)
-		)
-		(property "Datasheet" "~"
-			(at 215.9 130.81 0)
-			(effects
-				(font
-					(size 1.27 1.27)
-				)
-				(hide yes)
-			)
-		)
-		(property "Description" "Resistor, small symbol"
-			(at 215.9 130.81 0)
-			(effects
-				(font
-					(size 1.27 1.27)
-				)
-				(hide yes)
-			)
-		)
-		(pin "1"
-		)
-		(pin "2"
-		)
-		(instances
-			(project "test_battery"
-				(path "/21f56d4c-c23c-4f64-b5d5-a4783ab5b75c"
-					(reference "R11")
-					(unit 1)
-				)
