File: examples/ESP32S3/Lilka_v2/src/context/apps/batt_charger/module_resources/kicad_proj/batt_charger.kicad_sch (KiCad schematic)
At the start: 28 parts, among them J1 Lilka_PINS, J2 XL4016_IN, J3 XL4016_FB, J4 XL4016_OUT, Q1 A09T, Q2 A19T, Q3 A09T, Q4 A19T, Q5 A19T, Q6 A09T, Q7 A09T, U1 ADS1115IDGS, U2 INA219AxD

Commit message: fix example: в схему додано додаткову ємність
Parts:
- added C3: 20uF, Capacitor_SMD:C_1206_3216Metric_Pad1.33x1.80mm_HandSolder, symbol Device:C_Small
Connections:
- net 5V: now also C3.2
- net GND: now also C3.1
Changed lines of the file:
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@@
 	)
 	(junction
+		(at 237.49 123.19)
+		(diameter 0)
+		(color 0 0 0 0)
+	)
+	(junction
 		(at 116.84 154.94)
 		(diameter 0)
@@
 	(wire
 		(pts
+			(xy 237.49 123.19) (xy 237.49 135.89)
+		)
+		(stroke
+			(width 0)
+			(type default)
+		)
+	)
+	(wire
+		(pts
 			(xy 212.09 152.4) (xy 223.52 152.4)
 		)
@@
 	(wire
 		(pts
+			(xy 256.54 123.19) (xy 250.19 123.19)
+		)
+		(stroke
+			(width 0)
+			(type default)
+		)
+	)
+	(wire
+		(pts
 			(xy 247.65 71.12) (xy 229.87 71.12)
 		)
@@
 	(wire
 		(pts
-			(xy 237.49 129.54) (xy 237.49 135.89)
+			(xy 237.49 118.11) (xy 237.49 123.19)
 		)
 		(stroke
@@
 	(wire
 		(pts
+			(xy 256.54 127) (xy 256.54 123.19)
+		)
+		(stroke
+			(width 0)
+			(type default)
+		)
+	)
+	(wire
+		(pts
 			(xy 87.63 251.46) (xy 87.63 255.27)
 		)
@@
 	(wire
 		(pts
+			(xy 237.49 123.19) (xy 245.11 123.19)
+		)
+		(stroke
+			(width 0)
+			(type default)
+		)
+	)
+	(wire
+		(pts
 			(xy 106.68 154.94) (xy 116.84 154.94)
 		)
@@
 		(dnp no)
 		(fields_autoplaced yes)
-		(property "Reference" "#PWR10"
+		(property "Reference" "#PWR11"
 			(at 285.75 64.77 0)
 			(effects
@@
 			(project "batt_charger"
 				(path "/75962740-61ba-41b1-8e43-1d202dd04d24"
-					(reference "#PWR10")
+					(reference "#PWR11")
 					(unit 1)
 				)
@@
 	)
 	(symbol
+		(lib_id "power:GND")
+		(at 256.54 127 0)
+		(unit 1)
+		(exclude_from_sim no)
+		(in_bom yes)
+		(on_board yes)
+		(dnp no)
+		(fields_autoplaced yes)
+		(property "Reference" "#PWR10"
+			(at 256.54 133.35 0)
+			(effects
+				(font
+					(size 1.27 1.27)
+				)
+				(hide yes)
+			)
+		)
+		(property "Value" "GND"
+			(at 256.54 132.08 0)
+			(effects
+				(font
+					(size 1.27 1.27)
+				)
+			)
+		)
+		(property "Footprint" ""
+			(at 256.54 127 0)
+			(effects
+				(font
+					(size 1.27 1.27)
+				)
+				(hide yes)
+			)
+		)
+		(property "Datasheet" ""
+			(at 256.54 127 0)
+			(effects
+				(font
+					(size 1.27 1.27)
+				)
+				(hide yes)
+			)
+		)
+		(property "Description" "Power symbol creates a global label with name \"GND\" , ground"
+			(at 256.54 127 0)
+			(effects
+				(font
+					(size 1.27 1.27)
+				)
+				(hide yes)
+			)
+		)
+		(pin "1"
+		)
+		(instances
+			(project "batt_charger"
+				(path "/75962740-61ba-41b1-8e43-1d202dd04d24"
+					(reference "#PWR10")
+					(unit 1)
+				)
+			)
+		)
+	)
+	(symbol
 		(lib_id "Device:R_Small")
 		(at 96.52 130.81 90)
@@
 		(on_board yes)
 		(dnp no)
-		(property "Reference" "#PWR11"
+		(property "Reference" "#PWR14"
 			(at 309.88 64.77 0)
 			(effects
@@
 			(project "batt_charger"
 				(path "/75962740-61ba-41b1-8e43-1d202dd04d24"
-					(reference "#PWR11")
+					(reference "#PWR14")
 					(unit 1)
 				)
@@
 	(symbol
 		(lib_id "power:VCC")
-		(at 237.49 129.54 0)
+		(at 237.49 118.11 0)
 		(unit 1)
 		(exclude_from_sim no)
@@
 		(dnp no)
 		(property "Reference" "#PWR7"
-			(at 237.49 133.35 0)
+			(at 237.49 121.92 0)
 			(effects
 				(font
@@
 		)
 		(property "Value" "5V"
-			(at 237.49 125.222 0)
+			(at 237.49 113.792 0)
 			(effects
 				(font
@@
 		)
 		(property "Footprint" ""
-			(at 237.49 129.54 0)
+			(at 237.49 118.11 0)
 			(effects
 				(font
@@
 		)
 		(property "Datasheet" ""
-			(at 237.49 129.54 0)
+			(at 237.49 118.11 0)
 			(effects
 				(font
@@
 		)
 		(property "Description" "Power symbol creates a global label with name \"VCC\""
-			(at 237.49 129.54 0)
+			(at 237.49 118.11 0)
 			(effects
 				(font
@@
 		(on_board yes)
 		(dnp no)
-		(property "Reference" "#PWR13"
+		(property "Reference" "#PWR12"
 			(at 299.72 133.35 0)
 			(effects
@@
 			(project "batt_charger"
 				(path "/75962740-61ba-41b1-8e43-1d202dd04d24"
-					(reference "#PWR13")
+					(reference "#PWR12")
 					(unit 1)
 				)
@@
 		(dnp no)
 		(fields_autoplaced yes)
-		(property "Reference" "#PWR14"
+		(property "Reference" "#PWR13"
 			(at 299.72 179.07 0)
 			(effects
@@
 			(project "batt_charger"
 				(path "/75962740-61ba-41b1-8e43-1d202dd04d24"
-					(reference "#PWR14")
+					(reference "#PWR13")
 					(unit 1)
 				)
@@
 		(dnp no)
 		(fields_autoplaced yes)
-		(property "Reference" "#PWR12"
+		(property "Reference" "#PWR15"
 			(at 309.88 87.63 0)
 			(effects
@@
 			(project "batt_charger"
 				(path "/75962740-61ba-41b1-8e43-1d202dd04d24"
-					(reference "#PWR12")
+					(reference "#PWR15")
 					(unit 1)
 				)
@@
 					(unit 1)
 				)
+			)
+		)
+	)
+	(symbol
+		(lib_id "Device:C_Small")
+		(at 247.65 123.19 270)
+		(unit 1)
+		(exclude_from_sim no)
+		(in_bom yes)
+		(on_board yes)
+		(dnp no)
+		(fields_autoplaced yes)
+		(property "Reference" "C3"
+			(at 247.6436 116.84 90)
+			(effects
+				(font
+					(size 1.27 1.27)
+				)
+			)
+		)
+		(property "Value" "20uF"
+			(at 247.6436 119.38 90)
+			(effects
+				(font
+					(size 1.27 1.27)
+				)
+			)
+		)
+		(property "Footprint" "Capacitor_SMD:C_1206_3216Metric_Pad1.33x1.80mm_HandSolder"
+			(at 247.65 123.19 0)
+			(effects
+				(font
+					(size 1.27 1.27)
+				)
+				(hide yes)
+			)
+		)
+		(property "Datasheet" "~"
+			(at 247.65 123.19 0)
+			(effects
+				(font
+					(size 1.27 1.27)
+				)
+				(hide yes)
+			)
+		)
+		(property "Description" "Unpolarized capacitor, small symbol"
+			(at 247.65 123.19 0)
+			(effects
+				(font
+					(size 1.27 1.27)
+				)
+				(hide yes)
+			)
+		)
+		(pin "1"
+		)
+		(pin "2"
+		)
+		(instances
+			(project "batt_charger"
+				(path "/75962740-61ba-41b1-8e43-1d202dd04d24"
+					(reference "C3")
+					(unit 1)
+				)
